File: PicoLVDS.kicad_pcb (KiCad board)
At the start: 4 copper layers, 58 x 52.8 mm, 10 parts, among them J1 Conn_02x16, U1 Pico, U2 SN65LVDS047D, U3 SN65LVDS047D, U4 SN65LVDS047D, U5 SN65LVDS047D

Commit message: v2
Parts:
- U2, U3, U4, U5: value SN65LVDS047D -> SN65LVDS391D
- moved U5 0.11 mm to (47.7, 80.4)
Connections:
- U2 pad 11: /Out_1+ -> /Out_1-
- U2 pad 12: /Out_1- -> /Out_1+
- U2 pad 15: /Out_3+ -> /Out_3-
- U2 pad 16: /Out_3- -> /Out_3+
- U2 pad 8: GND -> +3V3
- U3 pad 11: /Out_5+ -> /Out_5-
- U3 pad 12: /Out_5- -> /Out_5+
- U3 pad 15: /Out_7+ -> /Out_7-
- U3 pad 16: /Out_7- -> /Out_7+
- U3 pad 8: GND -> +3V3
- U4 pad 11: /Out_9+ -> /Out_9-
- U4 pad 12: /Out_9- -> /Out_9+
- U4 pad 15: /Out_11+ -> /Out_11-
- U4 pad 16: /Out_11- -> /Out_11+
- U4 pad 8: GND -> +3V3
- U5 pad 11: /Out_13+ -> /Out_13-
- U5 pad 12: /Out_13- -> /Out_13+
- U5 pad 15: /Out_15+ -> /Out_15-
- U5 pad 16: /Out_15- -> /Out_15+
- U5 pad 8: GND -> +3V3
Routing:
- net GND: track 42.3 -> 36.5 mm, vias 12 -> 8
- net +3V3: track 16.6 -> 20.7 mm, vias 12 -> 16
- net /Out_6+: track 12.3 -> 13.3 mm
- net /Out_7+: track 13.0 -> 12.0 mm
- net /Out_11+: track 12.3 -> 13.2 mm
- net /Out_9+: track 12.3 -> 13.2 mm
- net /Out_3-: track 12.5 -> 13.3 mm
- net /Out_3+: track 12.6 -> 13.4 mm
- net /Out_8-: track 11.9 -> 12.7 mm
- net /Out_10-: track 12.5 -> 13.1 mm
- net /Out_14-: track 13.1 -> 12.5 mm
Other:
- board text added: "LVDS OUT"
- board text added: "PicoLVDS v2 Noah Paladino"
- board text removed: "SpinQuest DAQ Testbench v1 Noah Paladino"

Commit message: KiCad 9 Update
Other:
- board text added: "PicoLVDS v${REVISION} Noah Paladino"
- board text removed: "PicoLVDS v2 Noah Paladino"
