File: PicoLVDS.kicad_pcb (KiCad board)
At the start: 4 copper layers, 58 x 52.8 mm, 10 parts, among them J1 Conn_02x16, U1 Pico, U2 SN65LVDS391D, U3 SN65LVDS391D, U4 SN65LVDS391D, U5 SN65LVDS391D

Commit message: Schematic v2
Parts:
- added C5: C100n, Capacitor_SMD:C_0402_1005Metric_Pad0.74x0.62mm_HandSolder, F.Cu at (111.4, 63.8)
- added C6: C100n, Capacitor_SMD:C_0402_1005Metric_Pad0.74x0.62mm_HandSolder, F.Cu at (105.1, 63.8)
- added C7: C100n, Capacitor_SMD:C_0402_1005Metric_Pad0.74x0.62mm_HandSolder, F.Cu at (98.3, 63.8)
- added C8: C100n, Capacitor_SMD:C_0402_1005Metric_Pad0.74x0.62mm_HandSolder, F.Cu at (91.9, 63.8)
- added J2: RJHSE508002, RJHSE508002:AMPHENOL_RJHSE508002, F.Cu at (104.1, 47.8)
- added U10: SN65MLVD206BD, SN65MLVD206BD:D0008A_N, F.Cu at (114.6, 68.1)
- added U11: SN65MLVD206BD, SN65MLVD206BD:D0008A_N, F.Cu at (108.1, 68.1)
- added U8: SN65MLVD206BD, SN65MLVD206BD:D0008A_N, F.Cu at (101.5, 68.1)
- added U9: SN65MLVD206BD, SN65MLVD206BD:D0008A_N, F.Cu at (95.0, 68.1)
Connections:
- U1 pad 21: unconnected-(U1-GPIO16-Pad21)_1 -> /D16
- U1 pad 22: unconnected-(U1-GPIO17-Pad22)_1 -> /D17
- U1 pad 24: unconnected-(U1-GPIO18-Pad24) -> /D18
- U1 pad 25: unconnected-(U1-GPIO19-Pad25) -> /D19
- U1 pad 26: unconnected-(U1-GPIO20-Pad26) -> /SR
Routing:
- net /SR: track 0.00 -> 55.2 mm
- net /D16: track 0.00 -> 45.9 mm
- net /D17: track 0.00 -> 38.2 mm
- net /D18: track 0.00 -> 29.5 mm
- net /D19: track 0.00 -> 20.4 mm
- net GND: track 36.5 -> 22.0 mm, vias 8 -> 17
- net +3V3: track 20.7 -> 28.1 mm, vias 16 -> 20
- removed copper zone on F.Cu, net GND
Other:
- board size 58 x 52.8 mm -> 92.3 x 52.8 mm

Commit message: Switch to SMT footprint
Parts:
- U1: value Pico -> Raspberry Pi Pico 2; footprint RPi_Pico:RPi_Pico_SMD_TH -> RasPi_Pico:RasPi_Pico_2_SMD
- moved J2 6.10 mm to (104.1, 41.7)
Connections:
- net /Out_18+ renamed /RJ45_Out_18+
- net /Out_18- renamed /RJ45_Out_18-
- J2 pad 1_1: /Out_16+ -> /RJ45_Out_19-
- J2 pad 1_2: /Out_16- -> /RJ45_Out_19+
- J2 pad 1_3: /Out_17+ -> /RJ45_Out_17-
- J2 pad 1_6: /Out_17- -> /RJ45_Out_17+
- J2 pad 1_7: /Out_19+ -> /RJ45_Out_16-
- J2 pad 1_8: /Out_19- -> /RJ45_Out_16+
- J2 pad 2_1: /Out_16+ -> /RJ45_Out_19-
- J2 pad 2_2: /Out_16- -> /RJ45_Out_19+
- J2 pad 2_3: /Out_17+ -> /RJ45_Out_17-
- J2 pad 2_6: /Out_17- -> /RJ45_Out_17+
- J2 pad 2_7: /Out_19+ -> /RJ45_Out_16-
- J2 pad 2_8: /Out_19- -> /RJ45_Out_16+
- U10 pad 6: /Out_16+ -> /RJ45_Out_16+
- U10 pad 7: /Out_16- -> /RJ45_Out_16-
- U11 pad 6: /Out_17+ -> /RJ45_Out_17+
- U11 pad 7: /Out_17- -> /RJ45_Out_17-
- U9 pad 6: /Out_19+ -> /RJ45_Out_19+
- U9 pad 7: /Out_19- -> /RJ45_Out_19-
Routing:
- net /RJ45_Out_18+: track 0.00 -> 53.3 mm
- net /RJ45_Out_18-: track 0.00 -> 53.2 mm
- net /RJ45_Out_19-: track 0.00 -> 53.1 mm
- net /RJ45_Out_16-: track 0.00 -> 53.1 mm
- net /RJ45_Out_19+: track 0.00 -> 53.1 mm
- net /RJ45_Out_16+: track 0.00 -> 53.0 mm
- net /RJ45_Out_17+: track 0.00 -> 51.7 mm, vias 0 -> 1
- net /RJ45_Out_17-: track 0.00 -> 51.6 mm, vias 0 -> 1
- net /D19: track 20.4 -> 45.5 mm
- net /D18: track 29.5 -> 39.5 mm
- net /D17: track 38.2 -> 45.7 mm
- net GND: vias 17 -> 129
- net +3V3: vias 20 -> 36
- added copper zone on F.Cu, net +3V3
- added copper zone on F.Cu, net GND
- added copper zone on In2.Cu, net GND
