File: PicoLVDS.kicad_pcb (KiCad board)
At the start: 4 copper layers, 92.3 x 52.8 mm, 19 parts, among them J1 Conn_02x16, J2 RJHSE508002, U1 Raspberry Pi Pico 2, U10 SN65MLVD206BD, U11 SN65MLVD206BD, U2 SN65LVDS391D, U3 SN65LVDS391D, U4 SN65LVDS391D, U5 SN65LVDS391D, U8 SN65MLVD206BD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

Commit message: v3
Changed lines of the file:
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@@
 	)
 	(gr_text "PicoLVDS v${REVISION}\nNoah Paladino"
-		(at 41.6 62.8 90)
+		(at 102.87 80.772 0)
 		(layer "F.SilkS")
 		(effects
 			(font
 				(size 1.5 1.5)
-				(thickness 0.254)
+				(thickness 0.3)
 				(bold yes)
 			)
@@
 		(polygon
 			(pts
-				(xy 30 37.2) (xy 122.29 37.2) (xy 122.29 90) (xy 30 90)
+				(xy 30 37.2) (xy 83.312 37.338) (xy 83.312 62.484) (xy 122.174 62.484) (xy 122.29 90) (xy 30 90)
+			)
+		)
+	)
+	(zone
+		(net 2)
+		(net_name "GND")
+		(layer "In1.Cu")
+		(hatch edge 0.5)
+		(priority 2)
+		(connect_pads
+			(clearance 0.762)
+		)
+		(min_thickness 0.25)
+		(filled_areas_thickness no)
+		(fill yes
+			(thermal_gap 0.5)
+			(thermal_bridge_width 0.5)
+		)
+		(polygon
+			(pts
+				(xy 122.301 37.211) (xy 30.127 37.327) (xy 30.127 90.127) (xy 122.417 90.127)
 			)
 		)
